Commit message: Updates

File: iftomm_modified.urdf (robot description, URDF)
Before this commit: robot pulsar, 9 links, 8 joints
Links:
- link Link_0: mass 1.97 -> 0
- link Link_1: mass 1.97 -> 0
- link Link_2: mass 1.58 -> 0
- link Link_3: mass 1.17 -> 0
- link Link_EE: mass 2 -> 0
- link RW1: mass 4 -> 1
- link RW2: mass 4 -> 1
- link RW3: mass 4 -> 1
